Commit message: Obstacles simulated in gazebo

File: description/robot.urdf.xacro (robot description, xacro)
@@ -2,3 +2,4 @@
 <robot xmlns:xacro="http://www.ros.org/wiki/xacro"  name="robot">
     <xacro:include filename="robot_core.xacro" />
+    <xacro:include filename="/home/nsc9/dev_ws/src/herbie/description/gazebo_control.xacro" />
 </robot>

File: description/robot_core.xacro (robot description, xacro)
@@ -15,11 +15,12 @@
     </material>
     <!-- BASE LINK -->
-    <!-- CHASSIS LINK -->
     <link name="base_link">
     </link>
+    <!-- CHASSIS LINK -->
     <joint name="chassis_joint" type="fixed">
         <parent link="base_link"/>
         <child link="chassis"/>
         <origin xyz="-0.1 0 0"/>
+        <dynamics damping="0.05" friction="0.0"/>
     </joint>
     <link name="chassis">
@@ -41,4 +42,7 @@
         </xacro:inertial_box>
     </link>
+    <gazebo reference="chassis">
+        <material>Gazebo/White</material>
+    </gazebo>
     <!-- LEFT WHEEL LINK -->
     <joint name="left_wheel_joint" type="continuous">
@@ -47,4 +51,5 @@
         <origin xyz="0 0.175 0" rpy="-${pi/2} 0 0"/>
         <axis xyz="0 0 1"/>
+        <dynamics damping="0.05" friction="0.0"/>
     </joint>
     <link name="left_wheel">
@@ -64,4 +69,7 @@
         </xacro:inertial_cylinder>
     </link>
+    <gazebo reference="left_wheel">
+        <material>Gazebo/Blue</material>
+    </gazebo>
         <!-- RIGHT WHEEL LINK -->
     <joint name="right_wheel_joint" type="continuous">
@@ -70,4 +78,5 @@
         <origin xyz="0 -0.175 0" rpy="${pi/2} 0 0"/>
         <axis xyz="0 0 -1"/>
+        <dynamics damping="0.05" friction="0.0"/>
     </joint>
     <link name="right_wheel">
@@ -87,4 +96,7 @@
         </xacro:inertial_cylinder>
     </link>
+    <gazebo reference="right_wheel">
+        <material>Gazebo/Blue</material>
+    </gazebo>
     <!-- CASTER WHEEL LINK-->
     <joint name="caster_wheel_joint" type="fixed">
@@ -92,4 +104,5 @@
         <child link="caster_wheel"/>
         <origin xyz="0.24 0 0"/>
+        <dynamics damping="0.05" friction="0.0"/>
     </joint>
     <link name="caster_wheel">
@@ -110,3 +123,8 @@
         </xacro:inertial_sphere>
     </link>
+    <gazebo reference="caster_wheel">
+        <material>Gazebo/Black</material>
+        <mu1 value="0.001"/>
+        <mu2 value="0.001"/>
+    </gazebo>
 </robot>

Commit message: Added Lidar Camera

File: description/robot.urdf.xacro (robot description, xacro)
@@ -2,4 +2,6 @@
 <robot xmlns:xacro="http://www.ros.org/wiki/xacro"  name="robot">
     <xacro:include filename="robot_core.xacro" />
-    <xacro:include filename="/home/nsc9/dev_ws/src/herbie/description/gazebo_control.xacro" />
+    <xacro:include filename="/home/herbie/dev_ws/src/herbie/description/gazebo_control.xacro" />
+    <xacro:include filename="/home/herbie/dev_ws/src/herbie/description/lidar.xacro" />
+    <xacro:include filename="/home/herbie/dev_ws/src/herbie/description/camera.xacro" />
 </robot>

File: description/robot_core.xacro (robot description, xacro)
@@ -13,4 +13,7 @@
     <material name="black">
         <color rgba="0 0 0 1" />
+    </material>
+    <material name="red">
+        <color rgba="1 0 0 1"/>
     </material>
     <!-- BASE LINK -->
